Commit message: Fixed Joint name (L_wrist_yaw_joint)

File: 39-DoF/Wholebody_39_DoF_URDF/urdf/Wholebody_39_DoF_URDF.urdf (robot description, URDF)
Before this commit: robot Wholebody_39_DoF_URDF, 59 links, 58 joints
Links:
- added link world
Joints:
- removed joint L_wrist_yaw
- added joint L_wrist_yaw_joint: type revolute, parent L_elbow_pitch, child L_wrist_yaw, origin xyz=0 0 -0.13 rpy=0 0 0, axis 0 0 1, limit lower=-1.57 upper=1.57 effort=0 velocity=0
- added joint fixed_to_world: type fixed, parent world, child Pelvis, origin xyz=0 0 0.8582 rpy=0 0 0

Commit message: changed inertial values of the hand & wrist

File: 39-DoF/Wholebody_39_DoF_URDF/urdf/Wholebody_39_DoF_URDF.urdf (robot description, URDF)
Before this commit: robot Wholebody_39_DoF_URDF, 60 links, 59 joints
Links:
- link L_AA_1: mass 0.000901567166677004 -> 0.001
- link L_AA_2: mass 0.000901567166677004 -> 0.001
- link L_AA_3: mass 0.000901567166677003 -> 0.001
- link L_AA_4: mass 0.000901567166677003 -> 0.001
- link L_FE_1: mass 0.010491110414633 -> 0.01
- link L_FE_2: mass 0.0104903083657631 -> 0.01
- link L_FE_3: mass 0.0104902954833158 -> 0.01
- link L_FE_4: mass 0.0104902928738754 -> 0.01
- link L_FE_follower_1: mass 0.00704236095368229 -> 0.007
- link L_FE_follower_2: mass 0.00704211891368601 -> 0.007
- link L_FE_follower_3: mass 0.00704229670162109 -> 0.007
- link L_FE_follower_4: mass 0.00704232481737789 -> 0.007
- link L_elbow_pitch: mass 0.3055 -> 0.48
- link L_wrist_yaw: mass 0.395532703341776 -> 0.3392
- link R_AA_1: mass 0.000901567166677004 -> 0.001
- link R_AA_2: mass 0.000901567166677004 -> 0.001
- link R_AA_3: mass 0.000901567166677004 -> 0.001
- link R_AA_4: mass 0.000901567166677004 -> 0.001
- link R_FE_1: mass 0.010490303576979 -> 0.01
- link R_FE_2: mass 0.0104903083657632 -> 0.01
- link R_FE_3: mass 0.0104903113551846 -> 0.01
- link R_FE_4: mass 0.0104903072388752 -> 0.01
- link R_FE_follower_1: mass 0.00704239172409457 -> 0.007
- link R_FE_follower_2: mass 0.00704211842665845 -> 0.007
- link R_FE_follower_3: mass 0.00704238520387116 -> 0.007
- link R_FE_follower_4: mass 0.00704240684036434 -> 0.007
- link R_elbow_pitch: mass 0.304 -> 0.48
- link R_wrist_yaw: mass 0.395528663570662 -> 0.339200
Joints:
- joint L_elbow_pitch_joint: origin xyz=0 0 -0.0545 rpy=0 0 0 -> xyz=0 0 -0.0515 rpy=0 0 0
- joint L_wrist_yaw_joint: limit lower=-1.57 upper=1.57 effort=0 velocity=0 -> lower=-1.57 upper=1.57 effort=10 velocity=11.5
- joint R_elbow_pitch_joint: origin xyz=0 0 -0.0545 rpy=0 0 0 -> xyz=0 0 -0.0515 rpy=0 0 0
- joint R_wrist_yaw_joint: limit lower=-1.57 upper=1.57 effort=0 velocity=0 -> lower=-1.57 upper=1.57 effort=10 velocity=11.5

Commit message: fixed neck joint inertial values

File: 39-DoF/Wholebody_39_DoF_URDF/urdf/Wholebody_39_DoF_URDF.urdf (robot description, URDF)
Before this commit: robot Wholebody_39_DoF_URDF, 60 links, 59 joints
Links:
- link Neck_Pitch: mass 0.400888924681257 -> 0.433
- link Neck_Yaw: mass 0.061462 -> 0.108
